File: flip-clock.kicad_sch (KiCad schematic)
At the start: 9 parts, among them J1 Screw_Terminal_01x02, U1 ESP-01v090, U2 AP1117-33

Commit message: Added 3D models
Parts:
- J1: footprint TerminalBlock_RND:TerminalBlock_RND_205-00067_1x02_P7.50mm_Horizontal -> TerminalBlock_Phoenix:TerminalBlock_Phoenix_MKDS-1,5-2_1x02_P5.00mm_Horizontal
Connections:
- net at J1.1 (Pin_1): now also FL1.1; no longer FL1.3
- net at J1.2 (Pin_2): now also FL1.3; no longer FL1.1
Other:
- moved on the sheet: J1
Changed lines of the file:
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@@
     (pin "1")
   )
-  (symbol (lib_id "Connector:Screw_Terminal_01x02") (at 22.86 31.75 180) (unit 1)
+  (symbol (lib_id "Connector:Screw_Terminal_01x02") (at 22.86 29.21 0) (mirror y) (unit 1)
     (in_bom yes) (on_board yes) (fields_autoplaced)
     (property "Reference" "J1" (id 0) (at 24.892 24.5068 0))
     (property "Value" "Screw_Terminal_01x02" (id 1) (at 24.892 26.8055 0))
-    (property "Footprint" "TerminalBlock_RND:TerminalBlock_RND_205-00067_1x02_P7.50mm_Horizontal" (id 2) (at 22.86 31.75 0)
-      (effects (font (size 1.27 1.27)) hide)
-    )
-    (property "Datasheet" "~" (id 3) (at 22.86 31.75 0)
+    (property "Footprint" "TerminalBlock_Phoenix:TerminalBlock_Phoenix_MKDS-1,5-2_1x02_P5.00mm_Horizontal" (id 2) (at 22.86 29.21 0)
+      (effects (font (size 1.27 1.27)) hide)
+    )
+    (property "Datasheet" "~" (id 3) (at 22.86 29.21 0)
       (effects (font (size 1.27 1.27)) hide)
     )
@@
     )
     (path "/0049d02d-b2bd-4ae2-945f-14ed4f41e9f9"
-      (reference "J1") (unit 1) (value "Screw_Terminal_01x02") (footprint "TerminalBlock_RND:TerminalBlock_RND_205-00067_1x02_P7.50mm_Horizontal")
+      (reference "J1") (unit 1) (value "Screw_Terminal_01x02") (footprint "TerminalBlock_Phoenix:TerminalBlock_Phoenix_MKDS-1,5-2_1x02_P5.00mm_Horizontal")
     )
     (path "/b4e9ba94-1e48-4e68-ad99-460f09cc50a2"
